Commit message: fix ros_control and carrierbot_mapping

File: src/carrierbot_description/urdf/lidar.xacro (robot description, xacro)
@@ -1,13 +1,13 @@
 <?xml version="1.0"?>
 <robot xmlns:xacro="http://www.ros.org/wiki/xacro">
-    <xacro:property name="lidar_height" value="0.077" />
-    <xacro:property name="lidar_radius" value="0.039" />
+    <xacro:property name="lidar_height" value="0.037" />
+    <xacro:property name="lidar_radius" value="0.0345" />
     <!-- Include lidar -->
-    <link name="laser_link">
+    <link name="laser">
         <visual>
             <geometry>
                 <cylinder radius="${lidar_height}" length="${lidar_radius}" />
             </geometry>
-            <origin xyz="0 0 ${lidar_height/4}" rpy="0 0 0" />
+            <origin xyz="0 0 ${lidar_height/2 - 0.026}" rpy="0 0 0" />
             <material name="grey" />
         </visual>
@@ -22,6 +22,6 @@
     <joint name="laser_joint" type="fixed">
         <parent link="base_link" />
-        <child link="laser_link" />
-        <origin xyz="0 0 ${base_height}" rpy="0 0 0" />
+        <child link="laser" />
+        <origin xyz="${-base_length / 4.0} 0 ${base_height + 0.026}" rpy="0 0 0" />
     </joint>
     <gazebo reference="laser_link">
@@ -50,5 +50,5 @@
                 </ros>
                 <output_type>sensor_msgs/LaserScan</output_type>
-                <frame_name>laser_link</frame_name>
+                <frame_name>laser</frame_name>
             </plugin>
         </sensor>

File: src/carrierbot_description/urdf/mobile_base.xacro (robot description, xacro)
@@ -3,12 +3,12 @@
     <!--Dinamic
     var using xacro-->
-    <xacro:property name="base_length" value="0.7" />
-    <xacro:property name="base_width" value="0.75" />
-    <xacro:property name="base_height" value="0.2" />
-    <xacro:property name="wheel_radius" value="0.1" />
-    <xacro:property name="wheel_length" value="0.05" />
-    <xacro:property name="upper_base_length" value="0.4" />
-    <xacro:property name="upper_base_width" value="0.4" />
-    <xacro:property name="upper_base_height" value="0.8"/>
+    <xacro:property name="base_length" value="0.5" />
+    <xacro:property name="base_width" value="0.5" />
+    <xacro:property name="base_height" value="0.257" />
+    <xacro:property name="wheel_radius" value="0.0865" />
+    <xacro:property name="wheel_length" value="0.07" />
+    <xacro:property name="upper_base_length" value="0.21" />
+    <xacro:property name="upper_base_width" value="0.29" />
+    <xacro:property name="upper_base_height" value="1.064"/>
     <!-- Define links -->
     <link name="base_footprint" />
@@ -18,5 +18,5 @@
                 <box size="${base_length} ${base_width} ${base_height}" />
             </geometry>
-            <origin xyz="0 0 ${base_height/2.0}" rpy="0 0 0" />
+            <origin xyz="${-base_length / 4.0} 0 ${base_height/2.0}" rpy="0 0 0" />
             <material name="green" />
         </visual>
@@ -98,5 +98,5 @@
         <parent link="base_link" />
         <child link="right_wheel_link" />
-        <origin xyz="${-base_length / 4.0} ${-(base_width + wheel_length) / 2.0} 0" rpy="0 0 0" />
+        <origin xyz="0 ${-(base_width + wheel_length) / 2.0} 0" rpy="0 0 0" />
         <axis xyz="0 1 0" />
     </joint>
@@ -104,5 +104,5 @@
         <parent link="base_link" />
         <child link="left_wheel_link" />
-        <origin xyz="${-base_length / 4.0} ${(base_width + wheel_length) / 2.0} 0" rpy="0 0 0" />
+        <origin xyz="0 ${(base_width + wheel_length) / 2.0} 0" rpy="0 0 0" />
         <axis xyz="0 1 0" />
     </joint>
@@ -110,5 +110,5 @@
         <parent link="base_link" />
         <child link="caster_wheel_link" />
-        <origin xyz="${base_length / 3.0} 0 ${-wheel_radius / 2.0}" rpy="0 0 0" />
+        <origin xyz="${-base_length / 4.0 - base_length / 3.0} 0 ${-wheel_radius / 2.0}" rpy="0 0 0" />
         <axis xyz="0 1 0" />
     </joint>
@@ -116,5 +116,5 @@
         <parent link="base_link" />
         <child link="upper_base_link" />
-        <origin xyz="0 0 ${base_height + upper_base_height / 2.0}" rpy="0 0 0" />
+        <origin xyz="${-base_length / 4.0} 0 ${base_height + upper_base_height / 2.0}" rpy="0 0 0" />
     </joint>
 </robot>

File: src/carrierbot_description/urdf/my_robot.urdf.xacro (robot description, xacro)
@@ -8,4 +8,4 @@
   <xacro:include filename="ros2_control.xacro" />
   <!-- <xacro:include filename="camera.xacro" /> -->
-  <!-- <xacro:include filename="lidar.xacro"/> -->
+  <xacro:include filename="lidar.xacro"/>
 </robot>

File: src/carrierbot_description/urdf/ros2_control.xacro (robot description, xacro)
@@ -18,5 +18,5 @@
                 <plugin>carrierbot_firmware::CarrierbotInterface</plugin>
                 <param name="port">/dev/ttyUSB0</param>
-                <param name="baud_rate">115200</param>
+                <param name="baudrate">115200</param>
             </hardware>
         </xacro:unless>
