Commit message: add imu

File: src/carrierbot_description/urdf/my_robot.urdf.xacro (robot description, xacro)
@@ -8,4 +8,4 @@
   <xacro:include filename="ros2_control.xacro" />
   <!-- <xacro:include filename="camera.xacro" /> -->
-  <xacro:include filename="lidar.xacro"/>
+  <xacro:include filename="sensors.xacro"/>
 </robot>

File: src/carrierbot_description/urdf/sensors.xacro (robot description, xacro)
@@ -20,8 +20,30 @@
         </collision>
     </link>
+    <!-- Include IMU -->
+    <link name="imu">
+        <visual>
+            <geometry>
+                <box size="0.05 0.05 0.01" />
+            </geometry>
+            <origin xyz="0 0 0" rpy="0 0 0" />
+            <material name="grey" />
+        </visual>
+        <collision>
+            <geometry>
+                <box size="0.05 0.05 0.01" />
+            </geometry>
+            <origin xyz="0 0 0" rpy="0 0 0" />
+            <material name="grey" />
+        </collision>
+    </link>
     <joint name="laser_joint" type="fixed">
         <parent link="base_link" />
         <child link="laser" />
         <origin xyz="${-base_length / 4.0} 0 ${base_height + 0.026}" rpy="0 0 0" />
+    </joint>
+    <joint name="imu_joint" type="fixed">
+        <parent link="base_link" />
+        <child link="imu" />
+        <origin xyz="${-base_length / 4.0} 0 ${(base_height + 0.026) / 2.0}" rpy="0 0 0" />
     </joint>
     <gazebo reference="laser">
