Commit message: up

File: src/carrierbot_description/urdf/common_properties.xacro (robot description, xacro)
@@ -36,5 +36,5 @@
     </inertial>
   </xacro:macro>
-  <xacro:macro name="shpere_inertia" params="m r xyz rpy">
+  <xacro:macro name="sphere_inertia" params="m r xyz rpy">
     <inertial>
       <origin xyz="${xyz}" rpy="${rpy}" />

File: src/carrierbot_description/urdf/mobile_base.xacro (robot description, xacro)
@@ -86,5 +86,5 @@
             <origin xyz="0 0 0" rpy="0 0 0" />
         </collision>
-        <xacro:shpere_inertia m="5.0" r="${wheel_radius / 2.0}"
+        <xacro:sphere_inertia m="5.0" r="${wheel_radius / 2.0}"
             xyz="0 0 0" rpy="0 0 0" />
     </link>
