Commit message: up

File: src/carrierbot_description/urdf/mobile_base.xacro (robot description, xacro)
@@ -5,5 +5,5 @@
     <xacro:property name="base_length" value="0.5" />
     <xacro:property name="base_width" value="0.5" />
-    <xacro:property name="base_height" value="0.257" />
+    <xacro:property name="base_height" value="0.19" />
     <xacro:property name="wheel_radius" value="0.0865" />
     <xacro:property name="wheel_length" value="0.07" />
